File: SNES_logicadapter.kicad_sch (KiCad schematic)
At the start: 14 parts, among them CON1 SNES-CONN, CON2 SNES-CONN, J1 HP_1650-63203_logicanalyzer, J2 HP_1650-63203_logicanalyzer, J3 HP_1650-63203_logicanalyzer

Commit message: Auto-commit Fri Feb 17 21:15:47 EST 2023
Other:
- company: (none) -> matei repair lab
- title: (none) -> SNES logic adapter breakout / sniffer
Changed lines of the file:
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@@
 (kicad_sch (version 20211123) (generator eeschema)
   (paper "A4")
+  (title_block
+    (title "SNES logic adapter breakout / sniffer")
+    (date "2023-02-17")
+    (rev "1.0")
+    (company "matei repair lab")
+  )
   (junction (at 224.79 143.51) (diameter 0) (color 0 0 0 0)
   )
